File: KiCAD/PicoCAN.kicad_pcb (KiCad board)
At the start: 2 copper layers, 21 x 51.5 mm, 51 parts, among them J1 USB_C_Receptacle_USB2.0_14P, J2 Conn_01x20, J3 Conn_01x20, J4 Conn_01x02, J5 Screw_Terminal_01x03 (C381777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, J7 Conn_01x02, SW1 SW_Push, U1 RP2040, U2 MCP1700x-330xxTT, U3 W25Q16JVUXIQ, U4 MCP25625-x-SS (C481365), Y1 12 MHz Crystal_GND24 (C9002), Y2 16 MHz Crystal_GND24 (C13738)

Commit message: Finished Traces
Parts:
- added 5V: 5V TestPoint, TestPoint:TestPoint_Pad_1.0x1.0mm, F.Cu at (147.3, 119.2)
- moved R9 12.4 mm to (157.2, 113.0), turned to 0 degrees
- moved D2 12.0 mm to (157.5, 115.4)
- moved J4 10.5 mm to (158.6, 105.0)
- moved C21 9.54 mm to (147.4, 114.2), turned to -90 degrees
- moved SW1 8.95 mm to (157.2, 86.2), turned to 180 degrees
- moved C15 6.21 mm to (147.7, 103.0), turned to -90 degrees
- moved R5 5.48 mm to (153.2, 101.1), turned to 135 degrees
- moved R6 5.44 mm to (149.2, 85.1), turned to 180 degrees
- moved C16 5.21 mm to (153.3, 103.0), turned to 90 degrees
- moved C5 4.16 mm to (151.1, 85.9)
- moved C4 4.15 mm to (152.2, 85.9)
- moved C11 3.56 mm to (153.2, 88.0)
- moved C8 3.03 mm to (154.3, 104.5)
- moved U3 2.89 mm to (149.7, 88.5)
- moved C22 2.74 mm to (147.4, 116.3)
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Connections:
- C22 pad 1: +3V3 -> +5V
- J3 pad 11: RUN -> GPIO22
- J3 pad 12: GPIO22 -> RUN
- U4 pad : (no net) -> GND
- U4 pad 29: (no net) -> GND
Routing:
- net GND: track 0.00 -> 144.4 mm, vias 0 -> 26
- net +3V3: track 0.00 -> 123.5 mm, vias 0 -> 10
- net +5V: track 0.00 -> 76.0 mm, vias 0 -> 3
- net STBY: track 0.00 -> 47.2 mm, vias 0 -> 3
- net GPIO0: track 0.00 -> 44.0 mm, vias 0 -> 3
- net GPIO24: track 0.00 -> 34.3 mm, vias 0 -> 2
- net +1V1: track 0.00 -> 34.3 mm, vias 0 -> 3
- net GPIO2: track 0.00 -> 33.1 mm, vias 0 -> 2
- net GPIO3: track 0.00 -> 30.5 mm, vias 0 -> 2
- net VBUS: track 0.00 -> 27.4 mm, vias 0 -> 1
- net GPIO25: track 0.00 -> 27.2 mm, vias 0 -> 2
- net GPIO15: track 0.00 -> 27.1 mm, vias 0 -> 1
- net GPIO16: track 0.00 -> 26.1 mm
- net GPIO14: track 0.00 -> 24.7 mm, vias 0 -> 1
- net GPIO17: track 0.00 -> 22.7 mm
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- added copper zone on B.Cu, net GND
- added copper zone on F.Cu, net GND

Commit message: Finished PCB
Parts:
- C1 0: renamed from C10
- moved C7 0.09 mm to (147.2, 96.6)
- renumbered U3 to U
Routing:
- net GND: track 144.4 -> 148.8 mm, vias 26 -> 28
- net GPIO25: track 27.2 -> 28.8 mm
- net +5V: track 76.0 -> 74.5 mm
- net +3V3: track 123.5 -> 122.2 mm
- net GPIO24: track 34.3 -> 33.2 mm
Other:
- board text added: "0"
- board text added: "1"
- board text added: "10"
- board text added: "11"
- board text added: "12"
- board text added: "120Ω Term"
- board text added: "13"
- board text added: "14"
- board text added: "15"
- board text added: "16"
- board text added: "17"
- board text added: "18"
- board text added: "19"
- board text added: "2"
- board text added: "20"
- board text added: "21"
- board text added: "22"
- board text added: "24"
- board text added: "26"
- board text added: "27"
- board text added: "28"
- board text added: "29"
- board text added: "3"
- board text added: "3v3"
- board text added: "4"
- board text added: "5"
- board text added: "6"
- board text added: "7"
- board text added: "8"
- board text added: "9"
- board text added: "Built-in"
- board text added: "GND"
- board text added: "H"
- board text added: "INT"
- board text added: "L"
- board text added: "RUN"
- board text added: "STBY"
- board text added: "SWCLK"
- board text added: "SWD"
- board text added: "Term"
- board text added: "VBS"
- board text added: "VSYS"

Commit message: Finished PCB from earlier
Parts:
- C10: renamed from C1 0
- R1, R10, R11, R12, R2, R3, R4, R5, R6, R7, R8, R9: footprint LED_SMD:LED_0402_1005Metric -> Resistor_SMD:R_0402_1005Metric
- renumbered U to U3
Other:
- board text added: "C1"
- board text added: "U"
