File: KiCAD/PicoCAN.kicad_sch (KiCad schematic)
At the start: 52 parts, among them J1 USB_C_Receptacle_USB2.0_14P, J2 Conn_01x20, J3 Conn_01x20, J4 Conn_01x02, J5 Screw_Terminal_01x03 (C381777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, J7 Conn_01x02, SW1 SW_Push, U1 RP2040, U2 MCP1700x-330xxTT, U3 W25Q16JVUXIQ, U4 MCP25625-x-SS (C481365), Y1 12 MHz Crystal_GND24 (C9002), Y2 16 MHz Crystal_GND24 (C13738)

Commit message: Finished PCB from earlier
Parts:
- C1, C10: MPN (none) -> C52923
- C11, C12, C17, C2, C20, C21, C22, C3, C4, C5, C6, C7, C8, C9: MPN (none) -> C1525
- C13, C14: MPN (none) -> C96446
- C15, C16: MPN (none) -> C1562
- C18, C19: MPN (none) -> C1578; Notes (none) -> 10 pF: C32949
- D1: value C19171390 -> C2286; MPN (none) -> C2286
- D2: MPN (none) -> C2994781
- D3, D4: MPN (none) -> C223608
- J1: MPN (none) -> C165948
- J2, J3, J4, J7, TP1: now left out of the parts list
- J5: MPN (none) -> C3817776; Notes (none) -> Look at C3818779
- R1, R2: footprint LED_SMD:LED_0402_1005Metric -> Resistor_SMD:R_0402_1005Metric; MPN (none) -> C25905
- R10: footprint LED_SMD:LED_0402_1005Metric -> Resistor_SMD:R_0402_1005Metric; MPN (none) -> C25079
- R11, R12: footprint LED_SMD:LED_0402_1005Metric -> Resistor_SMD:R_0402_1005Metric; MPN (none) -> C25744
- R3, R4: value 27 -> 27R; footprint LED_SMD:LED_0402_1005Metric -> Resistor_SMD:R_0402_1005Metric; MPN (none) -> C25100
- R5, R7: footprint LED_SMD:LED_0402_1005Metric -> Resistor_SMD:R_0402_1005Metric; MPN (none) -> C11702
- R6: footprint LED_SMD:LED_0402_1005Metric -> Resistor_SMD:R_0402_1005Metric; MPN (none) -> C25744; Notes (none) -> Basic: C25744, Extended: C176114
- R8: footprint LED_SMD:LED_0402_1005Metric -> Resistor_SMD:R_0402_1005Metric; MPN (none) -> C25117
- R9: footprint LED_SMD:LED_0402_1005Metric -> Resistor_SMD:R_0402_1005Metric; MPN (none) -> C25076
- SW1: MPN (none) -> C720477
- U1: MPN (none) -> C2040
- U2: MPN (none) -> C39051
- U3: MPN (none) -> C2843335; Notes (none) -> Look at P25Q32L-UXH-IR later
- U4: MPN (none) -> C481365
- Y1: MPN (none) -> C9002
- Y2: MPN (none) -> C13738
